File: DasBlinkinput.kicad_pcb (KiCad board)
At the start: 2 copper layers, 0 parts

Commit message: First iteration of layout.
Parts:
- added C101: 1u, Capacitors_SMD:C_0805_HandSoldering, F.Cu at (124.7, 135.9)
- added C102: .1u, Capacitors_SMD:C_0805_HandSoldering, F.Cu at (134.1, 135.9)
- added C103: 100p, Capacitors_SMD:C_0805_HandSoldering, F.Cu at (132.4, 123.8)
- added C201: 100p, Capacitors_SMD:C_0805_HandSoldering, F.Cu at (147.1, 123.8)
- added C301: 100p, Capacitors_SMD:C_0805_HandSoldering, F.Cu at (162.1, 123.8)
- added C401: 100p, Capacitors_SMD:C_0805_HandSoldering, F.Cu at (172.5, 127.3)
- added P101: CONN_01X02, Pin_Headers:Pin_Header_Straight_1x02_Pitch2.00mm, F.Cu at (124.7, 139.7)
- added P102: CONN_01X05, Pin_Headers:Pin_Header_Straight_1x05_Pitch2.00mm, F.Cu at (158.5, 133.9)
- added PD101: QSB34CGR, gl:PD_QSB34, F.Cu at (124.8, 127.3)
- added PD201: QSB34CGR, gl:PD_QSB34, F.Cu at (139.6, 127.3)
- added PD301: QSB34CGR, gl:PD_QSB34, F.Cu at (154.3, 127.3)
- added PD401: QSB34CGR, gl:PD_QSB34, F.Cu at (169.0, 127.3)
- added R101: 0, Resistors_SMD:R_0805, F.Cu at (128.5, 138.9)
- added R102: 10k, Resistors_SMD:R_0805_HandSoldering, B.Cu at (136.9, 135.9)
- added R103: 10k, Resistors_SMD:R_0805_HandSoldering, B.Cu at (143.8, 132.3)
- added R104: 1M, Resistors_SMD:R_0805_HandSoldering, F.Cu at (132.3, 127.8)
- added R105: 10k, Resistors_SMD:R_0805_HandSoldering, B.Cu at (139.4, 135.9)
- added R106: 10k, Resistors_SMD:R_0805_HandSoldering, B.Cu at (151.9, 141.0)
- added R201: 1M, Resistors_SMD:R_0805_HandSoldering, F.Cu at (147.1, 127.8)
- added R301: 1M, Resistors_SMD:R_0805_HandSoldering, F.Cu at (162.1, 127.8)
- added R401: 1M, Resistors_SMD:R_0805_HandSoldering, F.Cu at (171.7, 136.1)
- added RV101: POT, gl:3296W_POT, F.Cu at (143.3, 138.4)
- added U101: MIC5501, TO_SOT_Packages_SMD:SOT-23-5, F.Cu at (128.5, 135.9)
- added U102: MCP6404, Housings_SOIC:SOIC-14_3.9x8.7mm_Pitch1.27mm, F.Cu at (164.8, 137.9)
- added U103: LM339, Housings_SOIC:SOIC-14_3.9x8.7mm_Pitch1.27mm, F.Cu at (151.9, 137.9)
- added W101: VGND, Connect:PINTST, F.Cu at (131.3, 130.8)
- added W102: GND, Connect:PINTST, F.Cu at (128.5, 141.7)
- added W103: +3v, Connect:PINTST, F.Cu at (131.6, 134.9)
- added W104: C, Connect:PINTST, F.Cu at (128.5, 127.8)
- added W105: REF, Connect:PINTST, F.Cu at (147.3, 142.5)
- added W201: C, Connect:PINTST, F.Cu at (143.5, 127.8)
- added W301: C, Connect:PINTST, F.Cu at (158.2, 127.8)
- added W401: C, Connect:PINTST, F.Cu at (170.4, 140.5)
Routing:
- net VGND: track 0.00 -> 70.5 mm, vias 0 -> 4
- net Net-(C103-Pad1): track 0.00 -> 54.6 mm, vias 0 -> 2
- net Net-(C103-Pad2): track 0.00 -> 53.7 mm, vias 0 -> 2
- net /+3v: track 0.00 -> 46.6 mm, vias 0 -> 5
- net Net-(C401-Pad1): track 0.00 -> 37.9 mm
- net Net-(C301-Pad1): track 0.00 -> 32.8 mm
- net GND: track 0.00 -> 32.5 mm, vias 0 -> 1
- net Net-(C201-Pad2): track 0.00 -> 30.6 mm
- net Net-(C201-Pad1): track 0.00 -> 30.5 mm
- net Net-(C301-Pad2): track 0.00 -> 27.8 mm
- net /Channel2/REF_IN: track 0.00 -> 24.1 mm
- net Net-(C401-Pad2): track 0.00 -> 23.0 mm
- net Net-(C101-Pad1): track 0.00 -> 7.47 mm
- net Net-(R105-Pad2): track 0.00 -> 5.48 mm
- net /Channel4/C_OUT: track 0.00 -> 5.45 mm
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- added copper zone on B.Cu, net GND
Other:
- board outline added: 51.6 x 22.1 mm

Commit message: Final board, with BOM.
Parts:
- added G***: LOGO, gl:ce-logo, B.Cu at (166.6, 128.3)
- C101: moved to B.Cu
- moved C101 4.59 mm to (128.5, 138.4), turned to 270 degrees
- moved P101 2.34 mm to (124.2, 137.4)
Routing:
- net GND: track 32.5 -> 24.8 mm
- net Net-(C101-Pad1): track 7.47 -> 10.1 mm
Other:
- board text added: "das-blinky-put"
